Commit message: reduce steer joint max vel

File: cob_test_rigs/robots/fdm/urdf/fdm.urdf.xacro (robot description, xacro)
@@ -7,4 +7,6 @@
   <!-- fdm -->
   <xacro:include filename="$(find cob_description)/urdf/drive_wheel/drive_wheel.urdf.xacro" />
+  <xacro:property name="drive_vel" value="19.95" />
+  <xacro:property name="steer_vel" value="12.00" /> <!-- Controller: 10.0, Driver: 12.0, Elmo: 15.0 -->
   <link name="world" />
   <!-- composition of the robot -->
